File: Christmas Tree.brd (EAGLE design)
At the start: 100 x 100 mm, 28 parts, among them J1 AVR_SPI_PROG_3X2NS, U1 ATTINY85-20SUR8S2-M

Commit message: update README
Parts:
- added U$1: XMASTREE, smd_leds:XMASTREE
- 10UF, C10, C11, C12, C13, C2, C3, C4, C5, C6, C7, C8, C9: device BeagleBone_Blue_R3:C0805 -> BeagleBone_Blue_R3:0805
Other:
- board text removed: "Learn how to program this at ThreeGirlsMakeStuff.com"
