File: Christmas Tree.sch (EAGLE design)
At the start: 28 parts, among them J1 AVR_SPI_PROG_3X2NS, U1 ATTINY85-20SUR8S2-M

Commit message: update README
Parts:
- added U$1: XMASTREE, smd_leds:XMASTREE
Other:
- moved on the sheet: CR2032, D1, J1, U$2
